Commit message: Add files via upload

File: dualarm_mobile_description/urdf/dualarm_mobile_description.urdf (robot description, URDF)
Before this commit: robot dualarm_mobile_description, 3 links, 2 joints
Joints:
- joint velodyne_front_joint: origin xyz=0.339947996689396 0.23499999999999 0.268200000000092 rpy=1.57079632679488 -1.7910313048242E-14 0.78539816339 -> xyz=0.339947996689396 0.23499999999999 0.268200000000092 rpy=1.57079632679488 -1.7910313048242E-14 -2.3561944902
